File: ESC_Board/ESC_BOARD_NEW.brd (EAGLE design)
At the start: 127 x 177.8 mm, 169 parts, among them J3 AVR_SPI_PROG_3X2NS, U2 ATMEGA328P_TQFP, U4 PCA9685

Commit message: God has abandoned us
Parts:
- turned C5 to 270 degrees
Routing:
- net PD3: track 0.00 -> 42.8 mm, vias 0 -> 1
- net PD6: track 0.00 -> 38.6 mm, vias 0 -> 1
- net PD4: track 0.00 -> 35.6 mm, vias 0 -> 2
- net PB0: track 0.00 -> 35.2 mm, vias 0 -> 2
- net PD5: track 0.00 -> 35.2 mm, vias 0 -> 1
- net PD7: track 0.00 -> 32.3 mm, vias 0 -> 2
- net +5V: track 87.6 -> 111.0 mm
- net MOSI: track 8.44 -> 18.3 mm
- net N$13: track 0.00 -> 6.19 mm
- net N$4: track 0.00 -> 6.19 mm
- net CUR2: track 7.80 -> 12.0 mm
- net CUR1: track 9.37 -> 13.6 mm
- net TEMP11: track 6.28 -> 10.5 mm
- net CUR6: track 6.38 -> 10.3 mm
- net CUR8: track 9.22 -> 13.2 mm
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
Commit message: There is light at the end of the tunnel
Parts:
- moved U$17 134.9 mm to (66.8, 4.06), turned to 90 degrees
- moved C10 118.2 mm to (20.8, 54.1)
- moved U$4 116.7 mm to (14.0, 55.1), turned to 180 degrees
- moved C66 109.6 mm to (5.08, 64.3), turned to 270 degrees
- moved C65 108.1 mm to (7.62, 64.3), turned to 270 degrees
- moved C64 106.6 mm to (10.2, 64.3), turned to 270 degrees
- moved C63 105.2 mm to (12.7, 64.3), turned to 270 degrees
- moved C25 104.1 mm to (180.1, 127.3)
- moved C26 104.1 mm to (180.1, 125.0)
- moved 12V-TO-5V1 104.1 mm to (175.8, 122.2)
- moved C24 104.1 mm to (170.4, 118.9)
- moved C62 103.9 mm to (15.2, 64.3), turned to 270 degrees
- moved C3 102.7 mm to (17.8, 64.3), turned to 270 degrees
- moved U$18 102.6 mm to (59.4, 44.2), turned to 90 degrees
- moved C2 101.6 mm to (20.3, 64.3), turned to 270 degrees
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Connections:
- net CUR10: now also U$4.CH5; no longer U$13.CH1
- net CUR11: now also U$13.CH4; no longer U$13.CH2
- net CUR3: now also U$13.CH0; no longer U$4.CH2
- net CUR4: now also U$13.CH1; no longer U$4.CH3
- net CUR5: now also U$4.CH2; no longer U$4.CH4
- net CUR6: now also U$4.CH3; no longer U$4.CH5
- net CUR7: now also U$13.CH2; no longer U$4.CH6
- net CUR8: now also U$13.CH3; no longer U$4.CH7
- net CUR9: now also U$4.CH4; no longer U$13.CH0
- net E1: now also U$4.CH6; no longer U$13.CH4
- net E2: now also U$4.CH7; no longer U$13.CH5
- net TEMP11: now also U$13.CH5; no longer U$13.CH3
Routing:
- net +5V: track 111.0 -> 147.3 mm, vias 4 -> 6
- net E4: track 13.9 -> 0.00 mm
- net CUR1: track 13.6 -> 0.00 mm
- net CUR8: track 13.2 -> 0.12 mm
- net E3: track 12.4 -> 0.00 mm
- net CUR2: track 12.0 -> 0.00 mm
- net CUR7: track 11.6 -> 0.00 mm
- net TEMP11: track 10.5 -> 0.00 mm
- net CUR9: track 10.4 -> 0.00 mm
- net CUR6: track 10.3 -> 0.00 mm
- net CUR3: track 10.3 -> 0.00 mm
- net E2: track 10.2 -> 0.00 mm
- net CUR10: track 9.91 -> 0.00 mm
- net CUR4: track 9.81 -> 0.00 mm
- net CUR5: track 9.81 -> 0.00 mm
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- added copper zone on layer 1, net ESC11
- added copper zone on layer 16, net ESC11
- added copper zone on layer 16, net N$63
- removed copper zone on layer 1, net +12V

Commit message: Thing and stuff done worked on
Parts:
- removed SV2: (no value), con-lsta:FE06-2
- moved P16 222.3 mm to (-48.5, 31.5), turned to 270 degrees
- moved P1 220.2 mm to (-48.5, 28.4), turned to 90 degrees
- moved P2 218.2 mm to (-48.5, 25.4), turned to 90 degrees
- moved P3 216.3 mm to (-48.5, 22.4), turned to 90 degrees
- moved P4 214.5 mm to (-48.5, 19.3), turned to 270 degrees
- moved P5 212.7 mm to (-48.5, 16.3), turned to 270 degrees
- moved P6 211.0 mm to (-48.5, 13.2), turned to 90 degrees
- moved ESC7_CON1 210.2 mm to (-45.2, -4.57), turned to 90 degrees
- moved ESC7_CON3 210.0 mm to (-36.6, -4.57), turned to 90 degrees
- moved ESC7_CON4 210.0 mm to (-28.2, -4.57), turned to 90 degrees
- moved P7 209.3 mm to (-48.5, 10.2), turned to 270 degrees
- moved C51 202.8 mm to (-38.9, 20.3), turned to 0 degrees
- moved R20 201.2 mm to (-38.9, 17.8), turned to 0 degrees
- moved R21 200.0 mm to (-38.9, 15.7), turned to 0 degrees
- moved R19 198.8 mm to (-38.9, 13.7), turned to 180 degrees
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Connections:
- removed net PWM0: P16.1, U4.6
- removed net PWM15: P15.1, U4.22
- new net PWME1: P6.1, U4.12
- new net PWME2: P7.1, U4.13
- net CS: no longer SV2.7
- net CUR1: now also U$4.CH3; no longer U$4.CH0
- net CUR10: now also U$4.CH0; no longer U$4.CH5
- net CUR2: now also U$4.CH2; no longer U$4.CH1
- net CUR5: now also U$4.CH4; no longer U$4.CH2
- net CUR6: now also U$4.CH1; no longer U$4.CH3
- net CUR9: now also U$4.CH5; no longer U$4.CH4
- net LED1: now also P13.1, U4.20; no longer P12.1, U4.19
- net LED2: now also P14.1, U4.21; no longer P13.1, U4.20
- net MISO: no longer SV2.9
- net MOSI: no longer SV2.8
- net PB0: no longer SV2.6
- net PD3: no longer SV2.2
- net PD4: no longer SV2.1
- net PD5: no longer SV2.3
- net PD6: no longer SV2.4
- net PD7: no longer SV2.5
- net PIEZO: now also P15.1, U4.22; no longer P14.1, U4.21
- net PWM1: now also P16.1, U4.6; no longer P1.1, U4.7
- net PWM10: now also P5.1, U4.11; no longer P10.1, U4.17
- net PWM11: now also P12.1, U4.19; no longer P11.1, U4.18
- net PWM2: now also P1.1, U4.7; no longer P2.1, U4.8
- net PWM3: now also P8.1, U4.15; no longer P3.1, U4.9
- net PWM4: now also P9.1, U4.16; no longer P4.1, U4.10
- net PWM5: now also P2.1, U4.8; no longer P5.1, U4.11
- net PWM6: now also P3.1, U4.9; no longer P6.1, U4.12
- net PWM7: no longer P7.1, U4.13
- net PWM8: now also P10.1, U4.17; no longer P8.1, U4.15
- net PWM9: now also P11.1, P4.1, U4.10, U4.18; no longer P9.1, U4.16
- net SCK: no longer SV2.10
- net SCL: no longer SV2.11
- net SDA: no longer SV2.12
Routing:
- net PWM2: track 17.2 -> 144.4 mm
- net CUR2: track 0.00 -> 118.7 mm, vias 0 -> 1
- net CUR1: track 0.00 -> 106.1 mm, vias 0 -> 3
- net PWM1: track 19.7 -> 118.7 mm
- net PWM6: track 8.18 -> 104.5 mm, vias 0 -> 1
- net CUR6: track 0.00 -> 78.7 mm, vias 0 -> 1
- net PWM5: track 9.62 -> 81.9 mm
- net CUR5: track 0.00 -> 68.8 mm, vias 0 -> 1
- net PWM10: track 8.47 -> 68.5 mm, vias 0 -> 1
- net PD3: track 42.8 -> 0.00 mm, vias 1 -> 0
- net PD6: track 38.6 -> 0.00 mm, vias 1 -> 0
- net CUR10: track 0.00 -> 38.5 mm, vias 0 -> 1
- net PIEZO: track 37.9 -> 0.00 mm
- net PD4: track 35.3 -> 0.00 mm, vias 2 -> 0
- net PB0: track 35.2 -> 0.00 mm, vias 2 -> 0
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- added copper zone on layer 1, net GND

Commit message: There is hope
Parts:
- removed P13, P14, P15: (no value), SparkFun-Connectors:1X01
- moved P8 162.3 mm to (125.0, 62.5)
- moved P9 158.4 mm to (121.9, 62.5)
- moved P10 154.6 mm to (118.9, 62.5)
- moved P11 150.7 mm to (115.8, 62.5)
- moved P12 147.0 mm to (112.8, 62.5)
- moved J5 93.1 mm to (19.6, 61.7), turned to 0 degrees
- moved J4 89.9 mm to (19.6, 58.7), turned to 0 degrees
- moved P16 73.6 mm to (17.3, 64.5)
- moved P1 72.4 mm to (14.2, 64.5)
- moved P2 71.4 mm to (11.2, 64.5)
- moved P3 70.6 mm to (8.13, 64.5)
- moved P4 70.1 mm to (5.08, 64.5)
- moved P5 69.9 mm to (2.03, 64.5)
- moved P6 62.7 mm to (5.08, 45.7)
- moved P7 61.8 mm to (2.03, 45.7)
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Connections:
- net CUR11: now also U$13.CH7; no longer U$13.CH4
- net CUR3: now also U$13.CH5; no longer U$13.CH0
- net CUR4: now also U$13.CH4; no longer U$13.CH1
- net CUR7: now also U$13.CH6; no longer U$13.CH2
- net E3: now also U$13.CH0; no longer U$13.CH6
- net E4: now also U$13.CH1; no longer U$13.CH7
- net LED1: no longer P13.1
- net LED2: no longer P14.1
- net PIEZO: no longer P15.1
- net PWM1: now also P5.1, U4.11; no longer P16.1, U4.6
- net PWM10: now also P16.1, U4.6; no longer P5.1, U4.11
- net PWM2: now also P4.1, U4.10; no longer P1.1, U4.7
- net PWM3: now also P9.1, U4.16; no longer P8.1, U4.15
- net PWM4: now also P8.1, U4.15; no longer P9.1, U4.16
- net PWM5: now also P3.1, U4.9; no longer P2.1, U4.8
- net PWM6: now also P2.1, U4.8; no longer P3.1, U4.9
- net PWM7: now also P11.1, U4.18
- net PWM9: now also P1.1, U4.7; no longer P11.1, P4.1, U4.10, U4.18
- net TEMP11: now also U$13.CH2; no longer U$13.CH5
Routing:
- net PWM3: track 0.00 -> 283.8 mm, vias 0 -> 1
- net PWM4: track 0.00 -> 262.8 mm, vias 0 -> 1
- net PWM7: track 0.00 -> 232.6 mm, vias 0 -> 2
- net PWM8: track 0.00 -> 216.4 mm, vias 0 -> 1
- net PWM11: track 0.00 -> 212.7 mm, vias 0 -> 1
- net CUR4: track 0.00 -> 106.5 mm, vias 0 -> 1
- net CUR3: track 0.00 -> 86.2 mm, vias 0 -> 5
- net CUR8: track 0.12 -> 67.0 mm, vias 0 -> 1
- net CUR7: track 0.00 -> 45.9 mm, vias 0 -> 1
- net PWM10: track 68.5 -> 104.3 mm
- net PWM9: track 42.7 -> 75.8 mm
- net PIEZO: track 0.00 -> 32.8 mm
- net PWM5: track 81.9 -> 113.7 mm
- net PWM6: track 104.5 -> 135.6 mm
- net PWM2: track 144.4 -> 175.0 mm
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- added copper zone on layer 1, net +12V

Commit message: More routing
Parts:
- moved C26 138.6 mm to (63.5, 50.0), turned to 90 degrees
- moved C25 137.9 mm to (65.8, 50.0), turned to 90 degrees
- moved 12V-TO-5V1 133.6 mm to (60.7, 54.4), turned to 270 degrees
- moved C24 131.9 mm to (57.9, 50.0)
- moved U$16 47.4 mm to (104.6, 44.5)
Routing:
- net +5V: track 141.1 -> 451.4 mm, vias 7 -> 20
- net TEMP11: track 15.2 -> 37.0 mm
- added copper zone on layer 1, net +5V

Commit message: This might actually work
Parts:
- moved RPI2 201.1 mm to (56.1, 16.8), turned to 270 degrees
- moved U$17 169.7 mm to (65.5, 173.7)
- moved C13 163.4 mm to (103.6, 7.11)
- moved C14 163.4 mm to (103.6, 9.65)
- moved C17 163.4 mm to (82.0, 4.83)
- moved Y2 163.4 mm to (85.9, 6.86)
- moved C12 163.4 mm to (84.3, 15.2)
- moved C15 163.4 mm to (86.9, 15.2)
- moved C16 163.4 mm to (82.0, 8.38)
- moved U2 163.4 mm to (95.5, 9.14)
- moved C11 154.4 mm to (146.6, 11.2)
- moved R10 154.4 mm to (146.6, 13.0)
- moved R38 154.4 mm to (152.7, 13.0)
- moved R39 154.4 mm to (152.7, 15.0)
- moved RESET 154.4 mm to (140.5, 11.9)
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Routing:
- net +5V: track 451.4 -> 576.9 mm, vias 20 -> 25
- net SCK: track 0.00 -> 60.4 mm
- net CS: track 0.00 -> 58.9 mm
- net MISO: track 6.62 -> 59.9 mm
- net MOSI: track 8.29 -> 59.3 mm
- net SCL: track 22.6 -> 0.00 mm, vias 1 -> 0
- net SDA: track 21.5 -> 0.00 mm, vias 1 -> 0
- net RESET: track 21.2 -> 0.00 mm, vias 2 -> 0
- net PIEZO: track 32.8 -> 24.9 mm, vias 0 -> 1
- net LED2: track 27.0 -> 20.0 mm, vias 0 -> 1
- net LED1: track 27.3 -> 20.9 mm, vias 0 -> 1
- net PWM4: track 262.8 -> 259.4 mm, vias 1 -> 0
- net +12V: track 2.29 -> 0.00 mm, vias 8 -> 11
- net PWM11: track 212.7 -> 214.7 mm, vias 1 -> 0
- net PWM3: track 283.8 -> 282.0 mm, vias 1 -> 0
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- added copper zone on layer 16, net GND

Commit message: GND is done messed up
Parts:
- moved J3 60.8 mm to (112.3, 11.9), turned to 270 degrees
- moved R39 50.9 mm to (103.4, 27.7), flipped to the bottom, turned to 270 degrees
- moved R38 49.0 mm to (105.9, 27.7), flipped to the bottom, turned to 270 degrees
- moved C11 25.1 mm to (121.7, 7.62), turned to 90 degrees
- moved R10 23.7 mm to (123.4, 7.62), turned to 270 degrees
- moved RESET 18.1 mm to (122.4, 13.7), turned to 270 degrees
- moved RPI2 7.95 mm to (52.6, 9.65), turned to 0 degrees
Connections:
- removed net SCL1: R21.1, U4.26
- removed net SDA1: R20.1, U4.27
- net SCL: now also R21.1, U4.26
- net SDA: now also R20.1, U4.27
Routing:
- net +5V: track 576.9 -> 602.2 mm, vias 25 -> 26
- net SCL1: track 4.47 -> 0.00 mm, vias 1 -> 0
- net SCL: track 0.00 -> 4.47 mm, vias 0 -> 1
- net SDA1: track 3.41 -> 0.00 mm, vias 1 -> 0
- net SDA: track 0.00 -> 3.41 mm, vias 0 -> 1

Commit message: Finishing up first layout of parts for ESC board
Parts:
- removed J4: (no value), SparkFun-Connectors:1X02
- removed R38, R39: (no value), SparkFun-Resistors:0603
- removed RPI2: T2I, BACKPLANE:T2I
- added C7, C8: 0.1uF, rcl:C0603
- added LED7, LED8: WS2812B5050, microbuilder:WS2812B
- moved C70 255.0 mm to (66.0, 19.3), flipped to the bottom, turned to 180 degrees
- moved C71 253.0 mm to (55.9, 19.1), flipped to the bottom, turned to 180 degrees
- moved LED2 246.6 mm to (41.1, 22.4), turned to 270 degrees
- moved LED1 228.4 mm to (34.3, 22.4), turned to 270 degrees
- moved C72 204.8 mm to (71.4, 15.7), flipped to the bottom, turned to 180 degrees
- moved LED6 197.7 mm to (72.6, 22.4), turned to 270 degrees
- moved LED3 188.4 mm to (48.0, 22.4), turned to 270 degrees
- moved C74 178.4 mm to (48.0, 17.3), turned to 270 degrees
- moved LED4 132.4 mm to (55.1, 22.4), turned to 270 degrees
- moved C73 130.5 mm to (41.1, 17.3), turned to 270 degrees
- moved LED5 121.8 mm to (66.0, 22.4), turned to 270 degrees
- moved C75 97.1 mm to (34.5, 17.3), turned to 270 degrees
- moved U$16 80.8 mm to (24.0, 32.4)
- moved R10 44.7 mm to (78.7, 8.76), flipped to the bottom
- moved RESET 43.4 mm to (79.5, 7.24), turned to 90 degrees
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Connections:
- removed net A0: U4.1
- removed net A1: U4.2
- removed net A2: U4.3
- removed net A3: U4.4
- removed net A4: U4.5
- removed net A5: U4.24
- removed net E2: J4.2, U$4.CH7
- removed net SCL_BRICKS: R38.1, U$16.P$12
- removed net SDA_BRICKS: R39.1, U$16.P$6
- new net OUT7: LED7.2-DOUT, LED8.4-DIN
- new net OUT8: LED8.2-DOUT
- net +12V: now also U$16.P$7, U$16.P$8, U$16.P$9; no longer U$16.P$1, U$16.P$2, U$16.P$3
- net +5V: now also C7.1, C8.1, LED7.1-VDD, LED8.1-VDD; no longer RPI2.3
- net 48_I_ANALOG: now also U$4.CH7
- net GND: now also C7.2, C8.2, LED7.3-GND, LED8.3-GND, U$16.P$1, U$16.P$2, U$16.P$3, U4.1, U4.2, U4.24, U4.3, U4.4, U4.5; no longer J4.1, RPI2.4, U$16.P$7, U$16.P$8, U$16.P$9
- net OUT6: now also LED7.4-DIN
- net SCL: now also U$16.P$12; no longer R38.2, RPI2.2
- net SDA: now also U$16.P$6; no longer R39.2, RPI2.1
Routing:
- net +5V: track 602.2 -> 766.0 mm, vias 26 -> 35
- net MOSI: track 59.3 -> 162.5 mm, vias 0 -> 2
- net CS: track 58.9 -> 161.6 mm, vias 0 -> 2
- net MISO: track 59.9 -> 155.1 mm, vias 0 -> 2
- net SCK: track 60.4 -> 154.4 mm, vias 0 -> 2
- net SDA: track 3.41 -> 65.3 mm, vias 1 -> 3
- net SCL: track 4.47 -> 63.9 mm, vias 1 -> 3
- net 48_I_ANALOG: track 0.00 -> 35.1 mm
- net RESET: track 0.00 -> 34.0 mm, vias 0 -> 2
- net PD3: track 0.00 -> 33.1 mm, vias 0 -> 2
- net OUT4: track 0.00 -> 18.1 mm, vias 0 -> 2
- net N$36: track 0.00 -> 8.96 mm
- net N$34: track 0.00 -> 8.96 mm
- net E2: track 8.89 -> 0.00 mm
- net N$35: track 0.00 -> 8.16 mm
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- removed copper zone on layer 1, net RESET
Other:
- board size 127 x 177.8 mm -> 127.7 x 178 mm
