File: ESC_Board/ESC_BOARD_NEW.sch (EAGLE design)
At the start: 187 parts, among them J3 AVR_SPI_PROG_3X2NS, U2 ATMEGA328P_TQFP, U4 PCA9685

Commit message: More layout stuff
Parts:
- removed C76, C77: 0.1uF, rcl:C-EUC0603
- removed LED7, LED8: WS2812B5050, microbuilder:WS2812B5050
Connections:
- removed net OUT7: LED7.DO, LED8.DI
- net +5V: no longer C76.1, C77.1, LED7.VDD, LED8.VDD
- net GND: no longer C76.2, C77.2, LED7.GND, LED8.GND
- net OUT3: no longer LED8.DO
- net OUT6: no longer LED7.DI
Changed lines of the file:
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@@
 <part name="GND109" library="supply1" library_urn="urn:adsk.eagle:library:371" deviceset="GND" device=""/>
 <part name="GND110" library="supply1" library_urn="urn:adsk.eagle:library:371" deviceset="GND" device=""/>
-<part name="LED7" library="microbuilder" deviceset="WS2812B5050" device="" value="WS2812B5050"/>
-<part name="C76" library="rcl" library_urn="urn:adsk.eagle:library:334" deviceset="C-EU" device="C0603" package3d_urn="urn:adsk.eagle:package:23616/2" value="0.1uF"/>
-<part name="P+41" library="supply1" library_urn="urn:adsk.eagle:library:371" deviceset="+5V" device=""/>
-<part name="GND111" library="supply1" library_urn="urn:adsk.eagle:library:371" deviceset="GND" device=""/>
-<part name="GND112" library="supply1" library_urn="urn:adsk.eagle:library:371" deviceset="GND" device=""/>
-<part name="LED8" library="microbuilder" deviceset="WS2812B5050" device="" value="WS2812B5050"/>
-<part name="C77" library="rcl" library_urn="urn:adsk.eagle:library:334" deviceset="C-EU" device="C0603" package3d_urn="urn:adsk.eagle:package:23616/2" value="0.1uF"/>
-<part name="P+42" library="supply1" library_urn="urn:adsk.eagle:library:371" deviceset="+5V" device=""/>
-<part name="GND113" library="supply1" library_urn="urn:adsk.eagle:library:371" deviceset="GND" device=""/>
-<part name="GND114" library="supply1" library_urn="urn:adsk.eagle:library:371" deviceset="GND" device=""/>
 <part name="P12" library="SparkFun-Connectors" deviceset="M01" device="PTH"/>
 <part name="P13" library="SparkFun-Connectors" deviceset="M01" device="PTH"/>
@@
 <part name="GND116" library="supply1" library_urn="urn:adsk.eagle:library:371" deviceset="GND" device=""/>
 <part name="GND117" library="supply1" library_urn="urn:adsk.eagle:library:371" deviceset="GND" device=""/>
-<part name="GND118" library="supply1" library_urn="urn:adsk.eagle:library:371" deviceset="GND" device=""/>
-<part name="GND119" library="supply1" library_urn="urn:adsk.eagle:library:371" deviceset="GND" device=""/>
 <part name="GND120" library="supply1" library_urn="urn:adsk.eagle:library:371" deviceset="GND" device=""/>
 <part name="GND121" library="supply1" library_urn="urn:adsk.eagle:library:371" deviceset="GND" device=""/>
@@
 <instance part="GND109" gate="1" x="297.18" y="139.7"/>
 <instance part="GND110" gate="1" x="287.02" y="144.78"/>
-<instance part="LED7" gate="G$1" x="340.36" y="134.62"/>
-<instance part="C76" gate="G$1" x="353.06" y="149.86"/>
-<instance part="P+41" gate="1" x="353.06" y="157.48"/>
-<instance part="GND111" gate="1" x="353.06" y="139.7"/>
-<instance part="GND112" gate="1" x="342.9" y="144.78"/>
-<instance part="LED8" gate="G$1" x="396.24" y="134.62"/>
-<instance part="C77" gate="G$1" x="408.94" y="149.86"/>
-<instance part="P+42" gate="1" x="408.94" y="157.48"/>
-<instance part="GND113" gate="1" x="408.94" y="139.7"/>
-<instance part="GND114" gate="1" x="398.78" y="144.78"/>
 <instance part="P12" gate="G$1" x="73.66" y="381" rot="MR0"/>
 <instance part="P13" gate="G$1" x="99.06" y="378.46" rot="MR0"/>
@@
 <instance part="GND116" gate="1" x="340.36" y="180.34"/>
 <instance part="GND117" gate="1" x="396.24" y="180.34"/>
-<instance part="GND118" gate="1" x="396.24" y="119.38"/>
-<instance part="GND119" gate="1" x="340.36" y="119.38"/>
 <instance part="GND120" gate="1" x="284.48" y="119.38"/>
 <instance part="GND121" gate="1" x="228.6" y="119.38"/>
@@
 </segment>
 <segment>
-<pinref part="C76" gate="G$1" pin="2"/>
-<wire x1="353.06" y1="144.78" x2="353.06" y2="142.24" width="0.1524" layer="91"/>
-<pinref part="GND111" gate="1" pin="GND"/>
-</segment>
-<segment>
-<pinref part="C77" gate="G$1" pin="2"/>
-<wire x1="408.94" y1="144.78" x2="408.94" y2="142.24" width="0.1524" layer="91"/>
-<pinref part="GND113" gate="1" pin="GND"/>
-</segment>
-<segment>
 <pinref part="GND121" gate="1" pin="GND"/>
 <pinref part="LED5" gate="G$1" pin="GND"/>
@@
 </segment>
 <segment>
-<pinref part="GND119" gate="1" pin="GND"/>
-<pinref part="LED7" gate="G$1" pin="GND"/>
-<wire x1="340.36" y1="121.92" x2="340.36" y2="124.46" width="0.1524" layer="91"/>
-</segment>
-<segment>
-<pinref part="GND118" gate="1" pin="GND"/>
-<pinref part="LED8" gate="G$1" pin="GND"/>
-<wire x1="396.24" y1="121.92" x2="396.24" y2="124.46" width="0.1524" layer="91"/>
-</segment>
-<segment>
 <pinref part="GND117" gate="1" pin="GND"/>
 <pinref part="LED4" gate="G$1" pin="GND"/>
@@
 <wire x1="297.18" y1="154.94" x2="297.18" y2="152.4" width="0.1524" layer="91"/>
 </segment>
-<segment>
-<pinref part="LED7" gate="G$1" pin="VDD"/>
-<wire x1="345.44" y1="149.86" x2="345.44" y2="152.4" width="0.1524" layer="91"/>
-<pinref part="C76" gate="G$1" pin="1"/>
-<wire x1="345.44" y1="152.4" x2="353.06" y2="152.4" width="0.1524" layer="91"/>
-<junction x="353.06" y="152.4"/>
-<pinref part="P+41" gate="1" pin="+5V"/>
-<wire x1="353.06" y1="154.94" x2="353.06" y2="152.4" width="0.1524" layer="91"/>
-</segment>
-<segment>
-<pinref part="LED8" gate="G$1" pin="VDD"/>
-<wire x1="401.32" y1="149.86" x2="401.32" y2="152.4" width="0.1524" layer="91"/>
-<pinref part="C77" gate="G$1" pin="1"/>
-<wire x1="401.32" y1="152.4" x2="408.94" y2="152.4" width="0.1524" layer="91"/>
-<junction x="408.94" y="152.4"/>
-<pinref part="P+42" gate="1" pin="+5V"/>
-<wire x1="408.94" y1="154.94" x2="408.94" y2="152.4" width="0.1524" layer="91"/>
-</segment>
 </net>
 <net name="N$2" class="0">
@@
 </segment>
 <segment>
-<pinref part="LED8" gate="G$1" pin="DO"/>
-<wire x1="421.64" y1="132.08" x2="408.94" y2="132.08" width="0.1524" layer="91"/>
-<label x="416.56" y="132.08" size="1.778" layer="95"/>
-</segment>
-<segment>
 <pinref part="LED4" gate="G$1" pin="DI"/>
 <wire x1="373.38" y1="195.58" x2="383.54" y2="195.58" width="0.1524" layer="91"/>
@@
 <label x="304.8" y="132.08" size="1.778" layer="95"/>
 </segment>
-<segment>
-<pinref part="LED7" gate="G$1" pin="DI"/>
-<wire x1="317.5" y1="132.08" x2="327.66" y2="132.08" width="0.1524" layer="91"/>
-<label x="317.5" y="132.08" size="1.778" layer="95"/>
-</segment>
-</net>
-<net name="OUT7" class="0">
-<segment>
-<pinref part="LED7" gate="G$1" pin="DO"/>
-<wire x1="365.76" y1="132.08" x2="353.06" y2="132.08" width="0.1524" layer="91"/>
-<label x="360.68" y="132.08" size="1.778" layer="95"/>
-</segment>
-<segment>
-<pinref part="LED8" gate="G$1" pin="DI"/>
-<wire x1="373.38" y1="132.08" x2="383.54" y2="132.08" width="0.1524" layer="91"/>
-<label x="373.38" y="132.08" size="1.778" layer="95"/>
-</segment>
 </net>

Commit message: Layout work
Parts:
- removed C53, C54, C55, C57, C58, C59, C60, C61, C7, C8, C9: 0.1uF, SparkFun-Capacitors:0.1UF-0603-25V-(+80/-20%)
- removed R22, R23, R24, R25, R28, R29, R30, R31, R32, R33, R34, R35, R36, R37, R4, R5, R6, R7, R8, R9: (no value), rcl:R-US_R0603
- removed U$14: MCP3008, MCP3008:MCP3008
- added ESC7_CON1, ESC7_CON3, ESC7_CON4: 3PINCONNECTOR, afro_20A_esc:3PINCONNECTOR
- added F1, F10, F11, F2, F3, F4, F5, F6, F7, F8, F9: 10A, PowerComponents:PTC(2920L)
- added J1, J2, J4, J5: (no value), SparkFun-Connectors:CONN_02
Connections:
- removed net ANALOG_6: U$14.CH6
- removed net N$52: U$14.CH7
- removed net PWM12: U4.PWM12
- removed net PWM13: P13.1, U4.PWM13
- removed net PWM14: P14.1, U4.PWM14
- removed net TEMP1: C57.1, R28.1, R29.2, U$4.CH0
- removed net TEMP10: C55.1, R24.1, R25.2, U$14.CH2
- removed net TEMP2: C58.1, R30.1, R31.2, U$4.CH2
- removed net TEMP3: C59.1, R32.1, R33.2, U$4.CH4
- removed net TEMP4: C60.1, R34.1, R35.2, U$4.CH6
- removed net TEMP5: C61.1, R36.1, R37.2, U$13.CH0
- removed net TEMP6: C7.1, R4.1, R5.2, U$13.CH2
- removed net TEMP7: C8.1, R6.1, R7.2, U$13.CH4
- removed net TEMP8: C9.1, R8.1, R9.2, U$13.CH6
- removed net TEMP9: C54.1, R22.1, R23.2, U$14.CH0
- new net E1: J5.2, U$13.CH4
- new net E2: J4.2, U$13.CH5
- new net E3: J1.2, U$13.CH6
- new net E4: J2.2, U$13.CH7
- new net LED1: ESC7_CON1.B, U4.PWM12
- new net LED2: ESC7_CON3.B, P13.1, U4.PWM13
- new net N$51: F6.1, U$7.IP1+, U$7.IP2+
- new net N$53: F1.1, U$1.IP1+, U$1.IP2+
- new net N$54: F2.1, U$2.IP1+, U$2.IP2+
- new net N$55: F3.1, U$3.IP1+, U$3.IP2+
- new net N$56: F4.1, U$5.IP1+, U$5.IP2+
- new net N$57: F5.1, U$6.IP1+, U$6.IP2+
- new net N$58: F7.1, U$8.IP1+, U$8.IP2+
- new net N$60: F8.1, U$9.IP1+, U$9.IP2+
- new net N$61: F9.1, U$10.IP1+, U$10.IP2+
- new net N$62: F10.1, U$11.IP1+, U$11.IP2+
- new net N$63: F11.1, U$12.IP1+, U$12.IP2+
- new net PIEZO: ESC7_CON4.B, P14.1, U4.PWM14
- net +12V: now also ESC7_CON1.C, ESC7_CON3.C, ESC7_CON4.C, F1.2, F10.2, F11.2, F2.2, F3.2, F4.2, F5.2, F6.2, F7.2, F8.2, F9.2; no longer U$1.IP1+, U$1.IP2+, U$10.IP1+, U$10.IP2+, U$11.IP1+, U$11.IP2+, U$12.IP1+, U$12.IP2+, U$2.IP1+, U$2.IP2+, U$3.IP1+, U$3.IP2+, U$5.IP1+, U$5.IP2+, U$6.IP1+, U$6.IP2+, U$7.IP1+, U$7.IP2+, U$8.IP1+, U$8.IP2+, U$9.IP1+, U$9.IP2+
- net +5V: no longer C53.1, R22.2, R24.2, R28.2, R30.2, R32.2, R34.2, R36.2, R4.2, R6.2, R8.2, U$14.VDD, U$14.VREF
- net CS: no longer U$14.CS/SHDN
- net CUR1: now also U$4.CH0; no longer U$4.CH1
- net CUR10: now also U$13.CH1; no longer U$14.CH3
- net CUR11: now also U$13.CH2; no longer U$14.CH5
- net CUR2: now also U$4.CH1; no longer U$4.CH3
- net CUR3: now also U$4.CH2; no longer U$4.CH5
- net CUR4: now also U$4.CH3; no longer U$4.CH7
- net CUR5: now also U$4.CH4; no longer U$13.CH1
- net CUR6: now also U$4.CH5; no longer U$13.CH3
- net CUR7: now also U$4.CH6; no longer U$13.CH5
- net CUR8: now also U$4.CH7; no longer U$13.CH7
- net CUR9: now also U$13.CH0; no longer U$14.CH1
- net GND: now also ESC7_CON1.A, ESC7_CON3.A, ESC7_CON4.A, J1.1, J2.1, J4.1, J5.1; no longer C53.2, C54.2, C55.2, C57.2, C58.2, C59.2, C60.2, C61.2, C7.2, C8.2, C9.2, R23.1, R25.1, R29.1, R31.1, R33.1, R35.1, R37.1, R5.1, R7.1, R9.1, U$14.AGND, U$14.DGND
- net MISO: no longer U$14.DOUT
- net MOSI: no longer U$14.DIN
- net SCK: no longer U$14.CLK
- net TEMP11: now also U$13.CH3; no longer U$14.CH4

Commit message: Initial layout
Connections:
- net LED1: now also P12.1
Changed lines of the file:
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@@
 <wire x1="55.88" y1="381" x2="66.04" y2="381" width="0.1524" layer="91"/>
 <label x="60.96" y="381" size="1.778" layer="95"/>
+<pinref part="P12" gate="G$1" pin="1"/>
 </segment>
 <segment>

Commit message: forgot schematic
Connections:
- net CUR10: now also U$4.CH5; no longer U$13.CH1
- net CUR11: now also U$13.CH4; no longer U$13.CH2
- net CUR3: now also U$13.CH0; no longer U$4.CH2
- net CUR4: now also U$13.CH1; no longer U$4.CH3
- net CUR5: now also U$4.CH2; no longer U$4.CH4
- net CUR6: now also U$4.CH3; no longer U$4.CH5
- net CUR7: now also U$13.CH2; no longer U$4.CH6
- net CUR8: now also U$13.CH3; no longer U$4.CH7
- net CUR9: now also U$4.CH4; no longer U$13.CH0
- net E1: now also U$4.CH6; no longer U$13.CH4
- net E2: now also U$4.CH7; no longer U$13.CH5
- net TEMP11: now also U$13.CH5; no longer U$13.CH3

Commit message: Thing and stuff done worked on
Parts:
- removed SV2: (no value), con-lsta:FE06-2
Connections:
- removed net PWM0: P16.1, U4.PWM0
- removed net PWM15: P15.1, U4.PWM15
- new net PWME1: P6.1, U4.PWM6
- new net PWME2: P7.1, U4.PWM7
- net CS: no longer SV2.7
- net CUR1: now also U$4.CH3; no longer U$4.CH0
- net CUR10: now also U$4.CH0; no longer U$4.CH5
- net CUR2: now also U$4.CH2; no longer U$4.CH1
- net CUR5: now also U$4.CH4; no longer U$4.CH2
- net CUR6: now also U$4.CH1; no longer U$4.CH3
- net CUR9: now also U$4.CH5; no longer U$4.CH4
- net LED1: now also P13.1, U4.PWM13; no longer P12.1, U4.PWM12
- net LED2: now also P14.1, U4.PWM14; no longer P13.1, U4.PWM13
- net MISO: no longer SV2.9
- net MOSI: no longer SV2.8
- net PB0: no longer SV2.6
- net PD3: no longer SV2.2
- net PD4: no longer SV2.1
- net PD5: no longer SV2.3
- net PD6: no longer SV2.4
- net PD7: no longer SV2.5
- net PIEZO: now also P15.1, U4.PWM15; no longer P14.1, U4.PWM14
- net PWM1: now also P16.1, U4.PWM0; no longer P1.1, U4.PWM1
- net PWM10: now also P5.1, U4.PWM5; no longer P10.1, U4.PWM10
- net PWM11: now also P12.1, U4.PWM12; no longer P11.1, U4.PWM11
- net PWM2: now also P1.1, U4.PWM1; no longer P2.1, U4.PWM2
- net PWM3: now also P8.1, U4.PWM8; no longer P3.1, U4.PWM3
- net PWM4: now also P9.1, U4.PWM9; no longer P4.1, U4.PWM4
- net PWM5: now also P2.1, U4.PWM2; no longer P5.1, U4.PWM5
- net PWM6: now also P3.1, U4.PWM3; no longer P6.1, U4.PWM6
- net PWM7: no longer P7.1, U4.PWM7
- net PWM8: now also P10.1, U4.PWM10; no longer P8.1, U4.PWM8
- net PWM9: now also P11.1, P4.1, U4.PWM11, U4.PWM4; no longer P9.1, U4.PWM9
- net SCK: no longer SV2.10
- net SCL: no longer SV2.11
- net SDA: no longer SV2.12
Other:
- note removed: "DEBUG PINS"

Commit message: There is hope
Parts:
- removed P13, P14, P15: (no value), SparkFun-Connectors:M01PTH
Connections:
- net CUR11: now also U$13.CH7; no longer U$13.CH4
- net CUR3: now also U$13.CH5; no longer U$13.CH0
- net CUR4: now also U$13.CH4; no longer U$13.CH1
- net CUR7: now also U$13.CH6; no longer U$13.CH2
- net E3: now also U$13.CH0; no longer U$13.CH6
- net E4: now also U$13.CH1; no longer U$13.CH7
- net LED1: no longer P13.1
- net LED2: no longer P14.1
- net PIEZO: no longer P15.1
- net PWM1: now also P5.1, U4.PWM5; no longer P16.1, U4.PWM0
- net PWM10: now also P16.1, U4.PWM0; no longer P5.1, U4.PWM5
- net PWM2: now also P4.1, U4.PWM4; no longer P1.1, U4.PWM1
- net PWM3: now also P9.1, U4.PWM9; no longer P8.1, U4.PWM8
- net PWM4: now also P8.1, U4.PWM8; no longer P9.1, U4.PWM9
- net PWM5: now also P3.1, U4.PWM3; no longer P2.1, U4.PWM2
- net PWM6: now also P2.1, U4.PWM2; no longer P3.1, U4.PWM3
- net PWM7: now also P11.1, U4.PWM11
- net PWM9: now also P1.1, U4.PWM1; no longer P11.1, P4.1, U4.PWM11, U4.PWM4
- net TEMP11: now also U$13.CH2; no longer U$13.CH5

Commit message: GND is done messed up
Connections:
- removed net SCL1: R21.1, U4.SCL
- removed net SDA1: R20.1, U4.SDA
- net SCL: now also R21.1, U4.SCL
- net SDA: now also R20.1, U4.SDA
Changed lines of the file:
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@@
 <label x="208.28" y="378.46" size="1.778" layer="95"/>
+</segment>
+<segment>
+<pinref part="U4" gate="G$1" pin="SDA"/>
+<wire x1="15.24" y1="406.4" x2="-5.08" y2="406.4" width="0.1524" layer="91"/>
+<pinref part="R20" gate="G$1" pin="1"/>
+<wire x1="-12.7" y1="401.32" x2="-5.08" y2="401.32" width="0.1524" layer="91"/>
+<wire x1="-5.08" y1="401.32" x2="-5.08" y2="406.4" width="0.1524" layer="91"/>
 </segment>
 </net>
@@
 <wire x1="274.32" y1="378.46" x2="292.1" y2="378.46" width="0.1524" layer="91"/>
 <label x="281.94" y="378.46" size="1.778" layer="95"/>
+</segment>
+<segment>
+<pinref part="U4" gate="G$1" pin="SCL"/>
+<wire x1="15.24" y1="403.86" x2="-2.54" y2="403.86" width="0.1524" layer="91"/>
+<pinref part="R21" gate="G$1" pin="1"/>
+<wire x1="-22.86" y1="398.78" x2="-2.54" y2="398.78" width="0.1524" layer="91"/>
+<wire x1="-2.54" y1="398.78" x2="-2.54" y2="403.86" width="0.1524" layer="91"/>
 </segment>
 </net>
@@
 </segment>
 </net>
-<net name="SCL1" class="0">
-<segment>
-<pinref part="U4" gate="G$1" pin="SCL"/>
-<wire x1="15.24" y1="403.86" x2="-2.54" y2="403.86" width="0.1524" layer="91"/>
-<pinref part="R21" gate="G$1" pin="1"/>
-<wire x1="-22.86" y1="398.78" x2="-2.54" y2="398.78" width="0.1524" layer="91"/>
-<wire x1="-2.54" y1="398.78" x2="-2.54" y2="403.86" width="0.1524" layer="91"/>
-</segment>
-</net>
-<net name="SDA1" class="0">
-<segment>
-<pinref part="U4" gate="G$1" pin="SDA"/>
-<wire x1="15.24" y1="406.4" x2="-5.08" y2="406.4" width="0.1524" layer="91"/>
-<pinref part="R20" gate="G$1" pin="1"/>
-<wire x1="-12.7" y1="401.32" x2="-5.08" y2="401.32" width="0.1524" layer="91"/>
-<wire x1="-5.08" y1="401.32" x2="-5.08" y2="406.4" width="0.1524" layer="91"/>
-</segment>
-</net>

Commit message: Finishing up first layout of parts for ESC board
Parts:
- removed J4: (no value), SparkFun-Connectors:CONN_02
- removed R38, R39: (no value), SparkFun-Resistors:RESISTOR0603
- removed RPI2: T2I, BACKPLANE:T2I
- added C7, C8: 0.1uF, rcl:C-EUC0603
- added LED7, LED8: WS2812B5050, microbuilder:WS2812B5050
Connections:
- removed net A0: U4.A0
- removed net A1: U4.A1
- removed net A2: U4.A2
- removed net A3: U4.A3
- removed net A4: U4.A4
- removed net A5: U4.A5
- removed net E2: J4.2, U$4.CH7
- removed net SCL_BRICKS: R38.1, U$16.P$12
- removed net SDA_BRICKS: R39.1, U$16.P$6
- new net OUT7: LED7.DO, LED8.DI
- new net OUT8: LED8.DO
- net +12V: now also U$16.P$7, U$16.P$8, U$16.P$9; no longer U$16.P$1, U$16.P$2, U$16.P$3
- net +5V: now also C7.1, C8.1, LED7.VDD, LED8.VDD; no longer RPI2.3
- net 48_I_ANALOG: now also U$4.CH7
- net GND: now also C7.2, C8.2, LED7.GND, LED8.GND, U$16.P$1, U$16.P$2, U$16.P$3, U4.A0, U4.A1, U4.A2, U4.A3, U4.A4, U4.A5; no longer J4.1, RPI2.4, U$16.P$7, U$16.P$8, U$16.P$9
- net OUT6: now also LED7.DI
- net SCL: now also U$16.P$12; no longer R38.2, RPI2.2
- net SDA: now also U$16.P$6; no longer R39.2, RPI2.1
